Commit message: temporal commit tested with real machine

File: mbzirc2020/mbzirc2020_task1/mbzirc2020_task1_common/robots/hydrus_only_rtkgps.urdf.xacro (robot description, xacro)
@@ -51,5 +51,5 @@
     <inertial>
       <origin xyz="0 0 0" rpy="0 0 0"/>
-      <mass value="0.06"/> <!-- plus center mounting bar 0.026 Kg -->
+      <mass value="${0.047 + 0.026}"/> <!-- plus center mounting bar 0.026 Kg -->
       <inertia
           ixx="0.0" iyy="0.0" izz="0.0"
@@ -57,4 +57,15 @@
     </inertial>
   </xacro:extra_module>
+  <xacro:extra_module name = "rtkgps_usb_cable" parent = "rtk_gps" visible = "0" >
+    <origin xyz="-0.13 0 0 " rpy="0 0 0"/>
+    <inertial>
+      <mass value = "0.017" />
+      <origin xyz="0 0 0" rpy="0 0 0"/>
+      <inertia
+          ixx="0.0" ixy="0.0" ixz="0.0"
+          iyy="0.0" iyz="0.0"
+          izz="0.0"/>
+    </inertial>
+  </xacro:extra_module>
   <!-- RTK GPS -->
 </robot>
